File: hardware/usb-power-switch.brd (EAGLE design)
At the start: 48.3 x 27.9 mm, 16 parts, among them IC1 TPS2024, IC2 LD1117V33

Commit message: Fixed several layout issues and removed unnecessary capacitor
Parts:
- removed C1: 0.1uF, rcl:C025-025X050
- R2, R3, R4, R5: device rcl:0204/7 -> rcl:0207/10
- moved C5 7.54 mm to (24.8, 19.1), turned to 90 degrees
- moved C4 5.08 mm to (24.8, 24.1), turned to 90 degrees
- moved JP2 2.54 mm to (47.0, 8.89)
- moved S1 2.23 mm to (39.1, 4.13), turned to 0 degrees
- moved R2 1.27 mm to (39.1, 15.2)
- moved R3 1.27 mm to (39.1, 13.0)
- moved R4 1.27 mm to (39.1, 10.8)
- moved R5 1.27 mm to (39.1, 8.57)
- moved OUT 0.16 mm to (18.9, 10.2)
Connections:
- net GND: now also S1.P$2; no longer C1.2, S1.P$3
- net GPIO0: now also S1.P$3; no longer S1.P$2
- net VIN: no longer C1.1
Routing:
- net /EN: track 32.3 -> 20.8 mm
- net RXI: track 17.1 -> 21.5 mm
- net VOUT: track 35.4 -> 38.1 mm
- net TXO: track 13.2 -> 15.8 mm
- net GPIO0: track 21.6 -> 24.1 mm
- net VCC: track 33.9 -> 34.8 mm, vias 0 -> 1
- net VIN: track 54.2 -> 53.5 mm
Other:
- board size 48.3 x 27.9 mm -> 50.8 x 27.9 mm
- board text added: "Wi-Fi USB Switch v2"
- board text removed: "Wi-Fi USB Switch v1"
