File: hardware/pcb/usb-power-switch.brd (EAGLE design)
At the start: 50.8 x 27.9 mm, 15 parts, among them IC1 TPS2024, IC2 LD1117V33

Commit message: Updated PCB to v3
Parts:
- removed C5: 10uF, rcl:C025-025X050
- removed IC1: TPS2024, ic-package:DIL08
- removed IC2: LD1117V33, SparkFun-PowerIC:78XXL
- removed JP1: ESP-01, pinhead:2X04
- removed JP2: FTDI 3.3V, pinhead:1X06
- removed R3, R4, R5: 10K, rcl:0207/10
- added C1: 22uF, rcl:C025-025X050
- added J1: ESP8266-01, pinhead:2X04
- added J2: FTDI 3.3V, pinhead:1X06
- added R1: 10K, rcl:0207/10
- added U$1: (no value), SparkFun-Aesthetics:OSHW-LOGO-S
- added U$2: (no value), SparkFun-Aesthetics:OSHW-LOGO-S_COPPER
- added U1: TPS2024, ic-package:DIL08
- added U2: LD1117V33, my-custom:TO-220
- C3: value 22uF -> 0.1uF
- C4: value 0.1uF -> 10uF
- IN: value USB-MINI-B -> WM17115-ND
- OUT: value USB-A -> UE27AC54100-ND
- S1: value TACTILE-BUTTON-MJTP1230 -> MJTP1230
- moved IN 57.5 mm to (57.4, 11.4), turned to 90 degrees
- moved C3 29.2 mm to (17.1, 4.45), turned to 180 degrees
- moved C4 19.8 mm to (22.2, 4.45), turned to 180 degrees
- moved C2 16.5 mm to (22.2, 18.4), turned to 0 degrees
- moved R2 13.6 mm to (30.8, 4.45)
- moved S1 9.27 mm to (33.3, 11.4), turned to 90 degrees
- moved OUT 8.82 mm to (10.2, 11.4), turned to 270 degrees
Connections:
- removed net CH_PD: JP1.3, R4.1
- removed net D+: IN.D+, OUT.P$3
- removed net D-: IN.D-, OUT.P$2
- removed net GPIO0: JP1.6, R3.1, S1.P$1, S1.P$3
- removed net RST: JP1.5, R5.1
- new net PU: J1.3, J1.5, J1.6, R2.1, S1.P$1, S1.P$3
- net /EN: now also J1.4, R1.1, U1.4; no longer IC1.4, JP1.4, R2.1
- net DTR: now also J2.6; no longer JP2.6
- net GND: now also C1.2, IN.GND1, IN.GND4, J1.2, J2.1, J2.2, OUT.P$5, OUT.P$6, U1.1, U2.P$1; no longer C3.2, C5.2, IC1.1, IC2.IN, JP1.2, JP2.1, JP2.2
- net RXI: now also J1.8, J2.4; no longer JP1.8, JP2.4
- net TXO: now also J1.1, J2.5; no longer JP1.1, JP2.5
- net VCC: now also C4.1, J1.7, R1.2, U2.P$2, U2.P$4; no longer C5.1, IC2.GND, JP1.7, R3.2, R4.2, R5.2
- net VIN: now also C3.1, J2.3, U1.2, U1.3, U2.P$3; no longer C4.1, IC1.2, IC1.3, IC2.OUT, JP2.3
- net VOUT: now also C1.1, U1.6, U1.7, U1.8; no longer C3.1, IC1.6, IC1.7, IC1.8
Routing:
- net VCC: track 34.8 -> 0.00 mm, vias 1 -> 0
- net GPIO0: track 24.1 -> 0.00 mm
- net VOUT: track 38.1 -> 14.1 mm
- net PU: track 0.00 -> 18.2 mm
- net D-: track 15.8 -> 0.00 mm
- net D+: track 14.8 -> 0.00 mm
- net RXI: track 21.5 -> 13.1 mm
- net /EN: track 20.8 -> 12.8 mm
- net CH_PD: track 7.80 -> 0.00 mm
- net TXO: track 15.8 -> 12.7 mm
- net RST: track 2.35 -> 0.00 mm
- net VIN: track 53.5 -> 54.8 mm
- added copper zone on layer 1, net VCC
Other:
- board size 50.8 x 27.9 mm -> 60.6 x 22.9 mm
- board text added: "WiFi USB V3"
- board text removed: "Prgm"
- board text removed: "Wi-Fi USB Switch v2"

Commit message: Optimized routing, added repo URL
Parts:
- moved U$1 0.38 mm to (53.1, 3.68)
- moved U$2 0.38 mm to (53.1, 3.68)
Connections:
- net /EN: now also R2.1; no longer R1.1
- net PU: now also R1.1; no longer R2.1
Routing:
- net /EN: track 12.8 -> 7.94 mm
- net PU: track 18.2 -> 18.9 mm
Other:
- board text added: "WiFi USB V3.1"
- board text added: "github.com/EPICmynamesBG/WiFi-USB"
- board text removed: "WiFi USB V3"
Changed lines of the file:
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@@
 <wire x1="60.579" y1="2.54" x2="60.579" y2="20.32" width="0.1524" layer="20"/>
 <wire x1="0" y1="20.32" x2="0" y2="2.54" width="0.1524" layer="20"/>
-<text x="52.705" y="18.542" size="1.4224" layer="21" ratio="15" distance="31" rot="R180" align="center">WiFi
+<text x="53.086" y="18.542" size="1.4224" layer="21" ratio="15" distance="31" rot="R180" align="center">WiFi
 USB
-V3</text>
+V3.1</text>
 <wire x1="2.54" y1="22.86" x2="58.039" y2="22.86" width="0.1524" layer="20"/>
 <circle x="24.892" y="6.223" radius="0.254" width="0.1524" layer="21"/>
@@
 <hole x="58.039" y="2.54" drill="2.794"/>
 <hole x="2.54" y="2.54" drill="2.794"/>
+<text x="40.64" y="20.32" size="1.016" layer="22" rot="MR0">github.com/EPICmynamesBG/WiFi-USB</text>
 </plain>
 <attributes>
@@
 <element name="J1" library="pinhead" package="2X04" value="ESP8266-01" x="27.559" y="11.43" smashed="yes" rot="R90"/>
 <element name="J2" library="pinhead" package="1X06" value="FTDI 3.3V" x="38.354" y="11.43" smashed="yes" rot="R90"/>
+<element name="R1" library="rcl" package="0207/10" value="10K" x="30.7975" y="18.415" smashed="yes">
+<attribute name="NAME" x="30.7975" y="19.5326" size="1.27" layer="25" ratio="10" rot="R180" align="top-center"/>
+</element>
 <element name="R2" library="rcl" package="0207/10" value="10K" x="30.7975" y="4.445" smashed="yes">
-<attribute name="NAME" x="30.7975" y="3.3274" size="1.27" layer="25" ratio="10" align="top-center"/>
-</element>
-<element name="R1" library="rcl" package="0207/10" value="10K" x="30.7975" y="18.415" smashed="yes">
-<attribute name="NAME" x="30.7975" y="19.558" size="1.27" layer="25" ratio="10" align="bottom-center"/>
+<attribute name="NAME" x="30.7975" y="3.302" size="1.27" layer="25" ratio="10" rot="R180" align="bottom-center"/>
 </element>
 <element name="S1" library="my-custom" package="TACTILE-BUTTON-MJTP1230" value="MJTP1230" x="33.3375" y="11.43" smashed="yes" rot="R90"/>
@@
 <attribute name="NAME" x="22.225" y="3.048" size="1.27" layer="25" ratio="10" rot="R180" align="bottom-center"/>
 </element>
-<element name="U$1" library="SparkFun-Aesthetics" package="OSHW-LOGO-S" value="" x="52.705" y="3.683"/>
-<element name="U$2" library="SparkFun-Aesthetics" package="OSHW-LOGO-S_COPPER" value="" x="52.705" y="3.683"/>
+<element name="U$1" library="SparkFun-Aesthetics" package="OSHW-LOGO-S" value="" x="53.086" y="3.683"/>
+<element name="U$2" library="SparkFun-Aesthetics" package="OSHW-LOGO-S_COPPER" value="" x="53.086" y="3.683"/>
 </elements>
 <signals>
@@
 </signal>
 <signal name="VCC">
-<contactref element="R2" pad="2"/>
+<contactref element="R1" pad="2"/>
 <contactref element="J1" pad="7"/>
 <contactref element="U2" pad="P$2"/>
-<contactref element="R1" pad="2"/>
+<contactref element="R2" pad="2"/>
 <contactref element="U2" pad="P$4"/>
 <contactref element="C4" pad="1"/>
@@
 <contactref element="J1" pad="5"/>
 <contactref element="J1" pad="3"/>
-<contactref element="R2" pad="1"/>
+<contactref element="R1" pad="1"/>
 <contactref element="S1" pad="P$3"/>
 <contactref element="S1" pad="P$1"/>
 <contactref element="J1" pad="6"/>
-<wire x1="28.829" y1="12.7" x2="30.809" y2="14.68" width="0.254" layer="1"/>
-<wire x1="30.809" y1="14.68" x2="31.0875" y2="14.68" width="0.254" layer="1"/>
-<wire x1="26.289" y1="12.7" x2="28.829" y2="12.7" width="0.254" layer="1"/>
-<wire x1="28.829" y1="12.7" x2="28.829" y2="10.16" width="0.254" layer="1"/>
-<wire x1="28.829" y1="10.16" x2="27.559" y2="8.89" width="0.254" layer="1"/>
-<wire x1="27.559" y1="8.89" x2="27.559" y2="6.2865" width="0.254" layer="1"/>
-<wire x1="27.559" y1="6.2865" x2="25.7175" y2="4.445" width="0.254" layer="1"/>
+<wire x1="26.289" y1="12.7" x2="28.829" y2="12.7" width="0.254" layer="16"/>
+<wire x1="28.829" y1="12.7" x2="28.829" y2="10.16" width="0.254" layer="16"/>
 <wire x1="28.829" y1="10.16" x2="29.1075" y2="10.16" width="0.254" layer="16"/>
 <wire x1="29.1075" y1="10.16" x2="31.0875" y2="8.18" width="0.254" layer="16"/>
+<wire x1="25.7175" y1="18.415" x2="27.2415" y2="16.891" width="0.254" layer="1"/>
+<wire x1="27.2415" y1="16.891" x2="30.099" y2="16.891" width="0.254" layer="1"/>
+<wire x1="30.099" y1="16.891" x2="31.0875" y2="15.9025" width="0.254" layer="1"/>
+<wire x1="31.0875" y1="15.9025" x2="31.0875" y2="14.68" width="0.254" layer="1"/>
+<wire x1="31.0875" y1="14.68" x2="29.1075" y2="12.7" width="0.254" layer="1"/>
+<wire x1="29.1075" y1="12.7" x2="28.829" y2="12.7" width="0.254" layer="1"/>
 </signal>
 <signal name="VIN">
@@
 <contactref element="U1" pad="4"/>
 <contactref element="J1" pad="4"/>
-<contactref element="R1" pad="1"/>
-<wire x1="23.495" y1="7.62" x2="26.035" y2="10.16" width="0.254" layer="1"/>
-<wire x1="26.035" y1="10.16" x2="26.289" y2="10.16" width="0.254" layer="1"/>
-<wire x1="25.7175" y1="18.415" x2="25.146" y2="17.8435" width="0.254" layer="1"/>
-<wire x1="25.146" y1="17.8435" x2="25.146" y2="11.303" width="0.254" layer="1"/>
-<wire x1="25.146" y1="11.303" x2="26.289" y2="10.16" width="0.254" layer="1"/>
+<contactref element="R2" pad="1"/>
+<wire x1="23.495" y1="7.62" x2="23.495" y2="6.6675" width="0.254" layer="1"/>
+<wire x1="23.495" y1="6.6675" x2="25.7175" y2="4.445" width="0.254" layer="1"/>
+<wire x1="23.495" y1="7.62" x2="26.035" y2="10.16" width="0.254" layer="16"/>
+<wire x1="26.035" y1="10.16" x2="26.289" y2="10.16" width="0.254" layer="16"/>
 </signal>
 <signal name="DTR">
